File: Eagle/mount.brd (EAGLE design)
At the start: 38 x 25 mm, 18 parts, among them U1 TINY45-20-DIP, X1 PAD6, X10 PAD4, X11 PAD4, X12 PAD4, X2 ZX62D-B-5PA8, X3 PAD6, X4 PAD2, X5 PAD2, X6 PAD2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

Commit message: Hello Egg
Connections:
- removed net DATA: SV1.4, U1.5, X4.P$1
- new net MOSI: SV1.4, U1.5
- net GND: now also X2.5; no longer X2.1
- net MISO: now also X4.P$1
- net N$6: now also X2.1; no longer X2.5
Routing:
- net DATA: track 21.8 -> 0.00 mm
- net MOSI: track 0.00 -> 17.1 mm
- net N$6: track 8.30 -> 0.00 mm
- net MISO: track 12.3 -> 16.4 mm
- net GND: track 25.0 -> 23.1 mm
Changed lines of the file:
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@@
 <grid distance="0.3175" unitdist="mm" unit="mm" style="lines" multiple="4" display="no" altdistance="0.15875" altunitdist="mm" altunit="mm"/>
 <layers>
-<layer number="1" name="Top" color="4" fill="1" visible="no" active="yes"/>
+<layer number="1" name="Top" color="4" fill="1" visible="yes" active="yes"/>
 <layer number="2" name="Route2" color="1" fill="3" visible="no" active="no"/>
 <layer number="3" name="Route3" color="4" fill="3" visible="no" active="no"/>
@@
 <layer number="14" name="Route14" color="1" fill="6" visible="no" active="no"/>
 <layer number="15" name="Route15" color="4" fill="6" visible="no" active="no"/>
-<layer number="16" name="Bottom" color="1" fill="1" visible="no" active="yes"/>
+<layer number="16" name="Bottom" color="1" fill="1" visible="yes" active="yes"/>
 <layer number="17" name="Pads" color="2" fill="1" visible="yes" active="yes"/>
-<layer number="18" name="Vias" color="2" fill="1" visible="no" active="yes"/>
-<layer number="19" name="Unrouted" color="6" fill="1" visible="no" active="yes"/>
+<layer number="18" name="Vias" color="2" fill="1" visible="yes" active="yes"/>
+<layer number="19" name="Unrouted" color="6" fill="1" visible="yes" active="yes"/>
 <layer number="20" name="Dimension" color="24" fill="1" visible="yes" active="yes"/>
 <layer number="21" name="tPlace" color="7" fill="10" visible="yes" active="yes"/>
@@
 <layer number="23" name="tOrigins" color="15" fill="1" visible="yes" active="yes"/>
 <layer number="24" name="bOrigins" color="15" fill="1" visible="no" active="yes"/>
-<layer number="25" name="tNames" color="7" fill="1" visible="yes" active="yes"/>
+<layer number="25" name="tNames" color="7" fill="1" visible="no" active="yes"/>
 <layer number="26" name="bNames" color="7" fill="1" visible="no" active="yes"/>
-<layer number="27" name="tValues" color="7" fill="1" visible="yes" active="yes"/>
+<layer number="27" name="tValues" color="7" fill="1" visible="no" active="yes"/>
 <layer number="28" name="bValues" color="7" fill="1" visible="no" active="yes"/>
 <layer number="29" name="tStop" color="7" fill="3" visible="no" active="yes"/>
@@
 <layer number="39" name="tKeepout" color="4" fill="11" visible="no" active="yes"/>
 <layer number="40" name="bKeepout" color="1" fill="11" visible="no" active="yes"/>
-<layer number="41" name="tRestrict" color="4" fill="10" visible="no" active="yes"/>
+<layer number="41" name="tRestrict" color="4" fill="10" visible="yes" active="yes"/>
 <layer number="42" name="bRestrict" color="1" fill="10" visible="no" active="yes"/>
 <layer number="43" name="vRestrict" color="2" fill="10" visible="no" active="yes"/>
 <layer number="44" name="Drills" color="7" fill="1" visible="no" active="yes"/>
-<layer number="45" name="Holes" color="7" fill="1" visible="no" active="yes"/>
+<layer number="45" name="Holes" color="7" fill="1" visible="yes" active="yes"/>
 <layer number="46" name="Milling" color="3" fill="1" visible="no" active="yes"/>
 <layer number="47" name="Measures" color="7" fill="1" visible="yes" active="yes"/>
@@
 <wire x1="11.1125" y1="4.7625" x2="11.1125" y2="4.8967" width="0.4064" layer="1"/>
 <via x="11.1125" y="4.8967" extent="1-16" drill="0.6"/>
-<contactref element="X2" pad="1"/>
 <contactref element="U1" pad="4"/>
 <wire x1="15.2875" y1="1.5875" x2="12.7" y2="1.5875" width="0.4064" layer="1"/>
@@
 <vertex x="9.2075" y="2.2225"/>
 </polygon>
-<wire x1="20.06" y1="20.19" x2="20.06" y2="18.675" width="0.4064" layer="1"/>
-<wire x1="20.06" y1="18.675" x2="20.32" y2="18.415" width="0.4064" layer="1"/>
 <contactref element="S1" pad="3"/>
 <contactref element="S2" pad="4"/>
+<contactref element="X2" pad="5"/>
+<wire x1="31.75" y1="15.9425" x2="26.5938" y2="23.2156" width="0" layer="19" extent="1-1"/>
+<wire x1="17.46" y1="20.19" x2="26.5938" y2="23.2156" width="0" layer="19" extent="1-1"/>
+<wire x1="14.9225" y1="15.875" x2="17.46" y2="20.19" width="0" layer="19" extent="1-1"/>
+<wire x1="11.1887" y1="23.2156" x2="17.46" y2="20.19" width="0" layer="19" extent="1-1"/>
+<wire x1="11.1125" y1="5.2317" x2="11.4275" y2="13.335" width="0" layer="19" extent="1-1"/>
+<wire x1="11.1125" y1="4.8967" x2="11.1125" y2="5.2317" width="0" layer="19" extent="1-1"/>
 </signal>
 <signal name="STROBE">
@@
 <wire x1="17.4625" y1="16.51" x2="19.05" y2="18.0975" width="0.4064" layer="16"/>
 <wire x1="19.05" y1="18.0975" x2="19.3675" y2="18.0975" width="0.4064" layer="16"/>
-</signal>
-<signal name="N$6">
-<contactref element="X2" pad="5"/>
-<contactref element="D1" pad="2"/>
-<wire x1="17.46" y1="20.19" x2="17.46" y2="18.095" width="0.4064" layer="1"/>
-<wire x1="17.46" y1="18.095" x2="16.8275" y2="17.4625" width="0.4064" layer="1"/>
-<wire x1="16.8275" y1="17.4625" x2="13.6525" y2="17.4625" width="0.4064" layer="1"/>
-<wire x1="12.319" y1="16.129" x2="12.319" y2="15.875" width="0.4064" layer="1"/>
-<wire x1="13.6525" y1="17.4625" x2="12.319" y2="16.129" width="0.4064" layer="1"/>
 </signal>
 <signal name="N$1">
@@
 <contactref element="SV1" pad="1"/>
 <wire x1="23.88" y1="13.4025" x2="26.67" y2="13.4025" width="0.4064" layer="16"/>
+<contactref element="X4" pad="P$1"/>
+<wire x1="16.14125" y1="4.7" x2="16.1925" y2="4.75125" width="0.4064" layer="1"/>
+<wire x1="16.1925" y1="6.985" x2="17.4625" y2="8.255" width="0.4064" layer="1"/>
+<wire x1="16.1925" y1="4.75125" x2="16.1925" y2="6.985" width="0.4064" layer="1"/>
 </signal>
 <signal name="CLOCK">
@@
 <wire x1="23.8125" y1="12.065" x2="20.0025" y2="8.255" width="0.4064" layer="16"/>
 </signal>
-<signal name="DATA">
-<contactref element="X4" pad="P$1"/>
-<contactref element="U1" pad="5"/>
-<wire x1="16.14125" y1="4.7" x2="16" y2="4.84125" width="0.4064" layer="1"/>
-<wire x1="16" y1="4.84125" x2="16" y2="5.25" width="0.4064" layer="1"/>
-<wire x1="16" y1="5.25" x2="15.9825" y2="6.8775" width="0.4064" layer="1"/>
-<wire x1="15.9825" y1="6.8775" x2="14.9225" y2="8.255" width="0.4064" layer="1"/>
+<signal name="MOSI">
 <contactref element="SV1" pad="4"/>
-<wire x1="14.9225" y1="8.255" x2="14.9225" y2="8.90625" width="0.4064" layer="1"/>
 <wire x1="14.9225" y1="8.90625" x2="18.24625" y2="12.23" width="0.4064" layer="1"/>
 <wire x1="22.25" y1="12.23" x2="24.7025" y2="14.6825" width="0.4064" layer="1"/>
@@
 <wire x1="27.7" y1="14.6825" x2="29.21" y2="15.9425" width="0.4064" layer="1"/>
 <wire x1="18.24625" y1="12.23" x2="22.25" y2="12.23" width="0.4064" layer="1"/>
+<contactref element="U1" pad="5"/>
+<wire x1="14.9225" y1="8.255" x2="14.9225" y2="8.90625" width="0" layer="19" extent="1-1"/>
 </signal>
 <signal name="N$5">
 <contactref element="X7" pad="P$1"/>
 </signal>
+<signal name="N$6">
+<contactref element="D1" pad="2"/>
+<contactref element="X2" pad="1"/>
+<wire x1="12.319" y1="15.875" x2="20.06" y2="20.19" width="0" layer="19" extent="1-1"/>
+</signal>
 </signals>
