File: Eagle/mount.sch (EAGLE design)
At the start: 18 parts, among them U1 TINY45-20-DIP, X1 PAD6, X10 PAD4, X11 PAD4, X12 PAD4, X2 ZX62D-B-5PA8, X3 PAD6, X4 PAD2, X5 PAD2, X6 PAD2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

Commit message: Hello Egg
Connections:
- removed net DATA: SV1.4, U1.PB0(MOSI), X4.P$1
- new net MOSI: SV1.4, U1.PB0(MOSI)
- net GND: now also X2G$1.5; no longer X2G$1.1
- net MISO: now also X4.P$1
- net N$6: now also X2G$1.1; no longer X2G$1.5
Other:
- note removed: "Die Buchse ist falsch nummeriert!"
Changed lines of the file:
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@@
 <sheet>
 <plain>
-<text x="12.7" y="76.2" size="1.778" layer="91">Die Buchse ist falsch nummeriert!</text>
 <text x="104.14" y="33.02" size="3.81" layer="94" ratio="10">ICSP</text>
 <frame x1="-10.16" y1="-10.16" x2="195.58" y2="134.62" columns="8" rows="5" layer="94"/>
 </plain>
 <instances>
-<instance part="X2" gate="G$1" x="35.56" y="88.9" rot="R270"/>
+<instance part="X2" gate="G$1" x="35.56" y="88.9" rot="MR270"/>
 <instance part="X1" gate="G$1" x="96.52" y="88.9"/>
 <instance part="X3" gate="G$1" x="96.52" y="83.82"/>
@@
 </segment>
 <segment>
-<pinref part="X2" gate="G$1" pin="1"/>
-<wire x1="40.64" y1="93.98" x2="40.64" y2="99.06" width="0.1524" layer="91"/>
 <pinref part="GND4" gate="1" pin="GND"/>
 <wire x1="40.64" y1="99.06" x2="55.88" y2="99.06" width="0.1524" layer="91"/>
 <wire x1="55.88" y1="99.06" x2="55.88" y2="81.28" width="0.1524" layer="91"/>
+<pinref part="X2" gate="G$1" pin="5"/>
+<wire x1="40.64" y1="99.06" x2="40.64" y2="93.98" width="0.1524" layer="91"/>
 </segment>
 <segment>
@@
 <wire x1="58.42" y1="35.56" x2="58.42" y2="50.8" width="0.1524" layer="91"/>
 <pinref part="S2" gate="1" pin="S"/>
-</segment>
-</net>
-<net name="N$6" class="0">
-<segment>
-<pinref part="X2" gate="G$1" pin="5"/>
-<pinref part="D1" gate="G$1" pin="AN"/>
-<wire x1="30.48" y1="96.52" x2="30.48" y2="93.98" width="0.1524" layer="91"/>
 </segment>
 </net>
@@
 <pinref part="U1" gate="G$1" pin="PB1(MISO)"/>
 <wire x1="81.28" y1="25.4" x2="81.28" y2="58.42" width="0.1524" layer="91"/>
-<wire x1="81.28" y1="58.42" x2="50.8" y2="58.42" width="0.1524" layer="91"/>
+<wire x1="81.28" y1="58.42" x2="63.5" y2="58.42" width="0.1524" layer="91"/>
 <pinref part="SV1" gate="1" pin="1"/>
+<pinref part="X4" gate="G$1" pin="P$1"/>
+<wire x1="63.5" y1="58.42" x2="50.8" y2="58.42" width="0.1524" layer="91"/>
+<wire x1="96.52" y1="71.12" x2="63.5" y2="71.12" width="0.1524" layer="91"/>
+<wire x1="63.5" y1="71.12" x2="63.5" y2="58.42" width="0.1524" layer="91"/>
+<label x="78.74" y="71.12" size="1.778" layer="95"/>
+<junction x="63.5" y="58.42"/>
 </segment>
 </net>
@@
 </segment>
 </net>
-<net name="DATA" class="0">
+<net name="MOSI" class="0">
 <segment>
 <wire x1="137.16" y1="22.86" x2="114.3" y2="22.86" width="0.1524" layer="91"/>
 <label x="127" y="22.86" size="1.778" layer="95"/>
 <wire x1="137.16" y1="22.86" x2="137.16" y2="40.64" width="0.1524" layer="91"/>
-<wire x1="137.16" y1="40.64" x2="73.66" y2="40.64" width="0.1524" layer="91"/>
-<pinref part="X4" gate="G$1" pin="P$1"/>
-<wire x1="96.52" y1="71.12" x2="73.66" y2="71.12" width="0.1524" layer="91"/>
-<wire x1="73.66" y1="71.12" x2="63.5" y2="71.12" width="0.1524" layer="91"/>
-<wire x1="63.5" y1="71.12" x2="63.5" y2="60.96" width="0.1524" layer="91"/>
+<wire x1="137.16" y1="40.64" x2="60.96" y2="40.64" width="0.1524" layer="91"/>
+<pinref part="SV1" gate="1" pin="4"/>
 <pinref part="U1" gate="G$1" pin="PB0(MOSI)"/>
-<wire x1="63.5" y1="60.96" x2="50.8" y2="60.96" width="0.1524" layer="91"/>
-<label x="78.74" y="71.12" size="1.778" layer="95"/>
-<wire x1="73.66" y1="40.64" x2="73.66" y2="71.12" width="0.1524" layer="91"/>
-<junction x="73.66" y="71.12"/>
-<pinref part="SV1" gate="1" pin="4"/>
+<wire x1="50.8" y1="60.96" x2="60.96" y2="60.96" width="0.1524" layer="91"/>
+<wire x1="60.96" y1="60.96" x2="60.96" y2="40.64" width="0.1524" layer="91"/>
 </segment>
 </net>
@@
 </segment>
 </net>
+<net name="N$6" class="0">
+<segment>
+<pinref part="D1" gate="G$1" pin="AN"/>
+<pinref part="X2" gate="G$1" pin="1"/>
+<wire x1="30.48" y1="96.52" x2="30.48" y2="93.98" width="0.1524" layer="91"/>
+</segment>
+</net>
